File: Hardware/Light Board/Hi-Light_ESP32-C3_MCU.kicad_sch (KiCad schematic)
At the start: 35 parts, among them U3 SPX3819M5-L-3-3, U4 ESP32-C3FH4X, Y1 40Mhz

Commit message: feat: Update board
Parts:
- R4: value 110R -> 10k
Changed lines of the file:
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@@
 			)
 		)
-		(property "Value" "110R"
+		(property "Value" "10k"
 			(at 107.188 175.26 0)
 			(effects
