File: Hardware/Light Board/HiLight.kicad_pcb (KiCad board)
At the start: 4 copper layers, 45 x 70 mm, 76 parts, among them J1 TYPE-C-31-M-12, J2 LED_CONN, J3 ENC_CONN, J4 UART_CONN, U1 USBLC6-2SC6, U2 TPS92360DCKR, U3 SPX3819M5-L-3-3, U4 ESP32-C3FH4X, Y1 40Mhz

Commit message: feat: Update board
Parts:
- R4: value 110R -> 10k
Changed lines of the file:
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@@
 			)
 		)
-		(property "Value" "110R"
+		(property "Value" "10k"
 			(at 0 1.17 270)
 			(layer "F.Fab")
